File: ESP32Board.sch (EAGLE design)
At the start: 20 parts, among them J1 MICRO_USB_B_HIROSE_ZX62-B-5PA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, U2 CH340K

Commit message: Fix connection
Parts:
- removed J1: MICRO_USB_B_HIROSE_ZX62-B-5PA(11), connector:MICRO_USB_B_HIROSE_ZX62-B-5PA(11)
- added J2: MICRO_USB_B_HIROSE_ZX62-B-5PA(11)MODEL, connector:MICRO_USB_B_HIROSE_ZX62-B-5PA(11)MODEL
- R4: value 2k -> 470
- R5: value 2k -> 1k
- renumbered GLED to LED, RLED to POWER
Connections:
- net GND: now also J2.GND; no longer J1.GND
- net UD+: now also J2.D+; no longer J1.D+
- net UD-: now also J2.D-; no longer J1.D-
- net USB5V: now also J2.+5V; no longer J1.+5V
Changed lines of the file:
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@@
 </classes>
 <parts>
-<part name="U$1" library="esp32" deviceset="ESP32-WROVER-E/ESP32-WROOM-32E" device=""/>
+<part name="U$1" library="esp32" library_urn="urn:adsk.eagle:library:33083408" deviceset="ESP32-WROVER-E/ESP32-WROOM-32E" device="" package3d_urn="urn:adsk.eagle:package:33083414/2"/>
 <part name="GND1" library="supply1" library_urn="urn:adsk.eagle:library:371" deviceset="GND" device=""/>
 <part name="GND2" library="supply1" library_urn="urn:adsk.eagle:library:371" deviceset="GND" device=""/>
@@
 <part name="C2" library="rcl" library_urn="urn:adsk.eagle:library:334" deviceset="C-EU" device="C0603K" package3d_urn="urn:adsk.eagle:package:23680/2" value="0.1µF"/>
 <part name="VDD1" library="supply1" library_urn="urn:adsk.eagle:library:371" deviceset="VDD" device=""/>
-<part name="J1" library="connector" deviceset="MICRO_USB_B_HIROSE_ZX62-B-5PA(11)" device=""/>
 <part name="GND4" library="supply1" library_urn="urn:adsk.eagle:library:371" deviceset="GND" device=""/>
 <part name="U2" library="CH340" deviceset="CH340K" device=""/>
@@
 <part name="GND8" library="supply1" library_urn="urn:adsk.eagle:library:371" deviceset="GND" device=""/>
 <part name="VDD3" library="supply1" library_urn="urn:adsk.eagle:library:371" deviceset="VDD" device=""/>
-<part name="R4" library="rcl" library_urn="urn:adsk.eagle:library:334" deviceset="R-US_" device="R0603" package3d_urn="urn:adsk.eagle:package:23555/3" value="2k"/>
-<part name="RLED" library="led" library_urn="urn:adsk.eagle:library:259" deviceset="LED" device="CHIPLED_0603" package3d_urn="urn:adsk.eagle:package:15822/2"/>
+<part name="R4" library="rcl" library_urn="urn:adsk.eagle:library:334" deviceset="R-US_" device="R0603" package3d_urn="urn:adsk.eagle:package:23555/3" value="470"/>
+<part name="POWER" library="led" library_urn="urn:adsk.eagle:library:259" deviceset="LED" device="CHIPLED_0603" package3d_urn="urn:adsk.eagle:package:15822/2"/>
 <part name="GND9" library="supply1" library_urn="urn:adsk.eagle:library:371" deviceset="GND" device=""/>
 <part name="C4" library="rcl" library_urn="urn:adsk.eagle:library:334" deviceset="C-EU" device="C0603K" package3d_urn="urn:adsk.eagle:package:23680/2" value="0.1µF"/>
 <part name="GND10" library="supply1" library_urn="urn:adsk.eagle:library:371" deviceset="GND" device=""/>
-<part name="GLED" library="led" library_urn="urn:adsk.eagle:library:259" deviceset="LED" device="CHIPLED_0603" package3d_urn="urn:adsk.eagle:package:15822/2"/>
+<part name="LED" library="led" library_urn="urn:adsk.eagle:library:259" deviceset="LED" device="CHIPLED_0603" package3d_urn="urn:adsk.eagle:package:15822/2"/>
 <part name="GND11" library="supply1" library_urn="urn:adsk.eagle:library:371" deviceset="GND" device=""/>
-<part name="R5" library="rcl" library_urn="urn:adsk.eagle:library:334" deviceset="R-US_" device="R0603" package3d_urn="urn:adsk.eagle:package:23555/3" value="2k"/>
+<part name="R5" library="rcl" library_urn="urn:adsk.eagle:library:334" deviceset="R-US_" device="R0603" package3d_urn="urn:adsk.eagle:package:23555/3" value="1k"/>
+<part name="J2" library="connector" deviceset="MICRO_USB_B_HIROSE_ZX62-B-5PA(11)" device="MODEL" package3d_urn="urn:adsk.eagle:package:6644353/2"/>
 </parts>
 <sheets>
@@
 <attribute name="VALUE" x="7.62" y="53.34" size="1.778" layer="96" rot="R90"/>
 </instance>
-<instance part="J1" gate="G$1" x="-81.28" y="53.34" smashed="yes" rot="R180">
-<attribute name="NAME" x="-76.2" y="44.45" size="1.778" layer="95" rot="R180"/>
-<attribute name="VALUE" x="-76.2" y="63.5" size="1.778" layer="95" rot="R180"/>
-</instance>
 <instance part="GND4" gate="1" x="-71.12" y="33.02" smashed="yes">
 <attribute name="VALUE" x="-73.66" y="30.48" size="1.778" layer="96"/>
@@
 <attribute name="VALUE" x="0.762" y="3.81" size="1.778" layer="96" rot="R90"/>
 </instance>
-<instance part="RLED" gate="G$1" x="-2.54" y="-2.54" smashed="yes">
+<instance part="POWER" gate="G$1" x="-2.54" y="-2.54" smashed="yes">
 <attribute name="NAME" x="1.016" y="-7.112" size="1.778" layer="95" rot="R90"/>
 <attribute name="VALUE" x="3.175" y="-7.112" size="1.778" layer="96" rot="R90"/>
@@
 <attribute name="VALUE" x="-15.24" y="33.02" size="1.778" layer="96"/>
 </instance>
-<instance part="GLED" gate="G$1" x="109.22" y="0" smashed="yes">
+<instance part="LED" gate="G$1" x="109.22" y="0" smashed="yes">
 <attribute name="NAME" x="112.776" y="-4.572" size="1.778" layer="95" rot="R90"/>
 <attribute name="VALUE" x="114.935" y="-4.572" size="1.778" layer="96" rot="R90"/>
@@
 <attribute name="NAME" x="107.7214" y="3.81" size="1.778" layer="95" rot="R90"/>
 <attribute name="VALUE" x="112.522" y="3.81" size="1.778" layer="96" rot="R90"/>
+</instance>
+<instance part="J2" gate="G$1" x="-81.28" y="53.34" smashed="yes" rot="R180">
+<attribute name="NAME" x="-76.2" y="44.45" size="1.778" layer="95" rot="R180"/>
+<attribute name="VALUE" x="-76.2" y="63.5" size="1.778" layer="95" rot="R180"/>
 </instance>
 </instances>
@@
 <pinref part="U2" gate="G$1" pin="GND"/>
 <wire x1="-55.88" y1="55.88" x2="-71.12" y2="55.88" width="0.1524" layer="91"/>
-<pinref part="J1" gate="G$1" pin="GND"/>
 <wire x1="-73.66" y1="58.42" x2="-71.12" y2="58.42" width="0.1524" layer="91"/>
 <wire x1="-71.12" y1="58.42" x2="-71.12" y2="55.88" width="0.1524" layer="91"/>
 <junction x="-71.12" y="55.88"/>
+<pinref part="J2" gate="G$1" pin="GND"/>
 </segment>
 <segment>
@@
 </segment>
 <segment>
-<pinref part="RLED" gate="G$1" pin="C"/>
+<pinref part="POWER" gate="G$1" pin="C"/>
 <pinref part="GND9" gate="1" pin="GND"/>
 </segment>
@@
 </segment>
 <segment>
-<pinref part="GLED" gate="G$1" pin="C"/>
+<pinref part="LED" gate="G$1" pin="C"/>
 <pinref part="GND11" gate="1" pin="GND"/>
 </segment>
@@
 <segment>
 <pinref part="U2" gate="G$1" pin="UD+"/>
-<pinref part="J1" gate="G$1" pin="D+"/>
 <wire x1="-55.88" y1="53.34" x2="-73.66" y2="53.34" width="0.1524" layer="91"/>
 <label x="-63.5" y="53.34" size="1.778" layer="95"/>
+<pinref part="J2" gate="G$1" pin="D+"/>
 </segment>
 </net>
 <net name="UD-" class="0">
 <segment>
-<pinref part="J1" gate="G$1" pin="D-"/>
 <pinref part="U2" gate="G$1" pin="UD-"/>
 <wire x1="-73.66" y1="50.8" x2="-55.88" y2="50.8" width="0.1524" layer="91"/>
 <label x="-63.5" y="50.8" size="1.778" layer="95"/>
+<pinref part="J2" gate="G$1" pin="D-"/>
 </segment>
 </net>
@@
 <wire x1="-12.7" y1="68.58" x2="-68.58" y2="68.58" width="0.1524" layer="91"/>
 <wire x1="-68.58" y1="68.58" x2="-68.58" y2="48.26" width="0.1524" layer="91"/>
-<pinref part="J1" gate="G$1" pin="+5V"/>
 <wire x1="-68.58" y1="48.26" x2="-73.66" y2="48.26" width="0.1524" layer="91"/>
 <label x="-66.04" y="68.58" size="1.778" layer="95"/>
@@
 <junction x="-12.7" y="48.26"/>
 <pinref part="C4" gate="G$1" pin="1"/>
+<pinref part="J2" gate="G$1" pin="+5V"/>
 </segment>
 </net>
@@
 <wire x1="-35.56" y1="-33.02" x2="-27.94" y2="-33.02" width="0.1524" layer="91"/>
 <pinref part="R3" gate="G$1" pin="1"/>
-<wire x1="-27.94" y1="-33.02" x2="-20.32" y2="-33.02" width="0.1524" layer="91"/>
 <wire x1="-27.94" y1="-30.48" x2="-27.94" y2="-33.02" width="0.1524" layer="91"/>
 <junction x="-27.94" y="-33.02"/>
 <wire x1="-27.94" y1="-33.02" x2="-27.94" y2="-35.56" width="0.1524" layer="91"/>
 <pinref part="C7" gate="G$1" pin="1"/>
-<label x="-20.32" y="-33.02" size="1.778" layer="95" xref="yes"/>
+<label x="-10.16" y="-33.02" size="1.778" layer="95" xref="yes"/>
+<wire x1="-27.94" y1="-33.02" x2="-10.16" y2="-33.02" width="0.1524" layer="91"/>
 </segment>
 </net>
@@
 <segment>
 <pinref part="R4" gate="G$1" pin="1"/>
-<pinref part="RLED" gate="G$1" pin="A"/>
+<pinref part="POWER" gate="G$1" pin="A"/>
 </segment>
 </net>
@@
 <net name="N$1" class="0">
 <segment>
-<pinref part="GLED" gate="G$1" pin="A"/>
+<pinref part="LED" gate="G$1" pin="A"/>
 <pinref part="R5" gate="G$1" pin="1"/>
 </segment>

Commit message: Add reset switch
Parts:
- added U$2: TVAF06-A020B-R, switches:TVAF06-A020B-R
Connections:
- net EN: now also U$2.A
- net GND: now also U$2.B
Changed lines of the file:
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@@
 <part name="R5" library="rcl" library_urn="urn:adsk.eagle:library:334" deviceset="R-US_" device="R0603" package3d_urn="urn:adsk.eagle:package:23555/3" value="1k"/>
 <part name="J2" library="connector" deviceset="MICRO_USB_B_HIROSE_ZX62-B-5PA(11)" device="MODEL" package3d_urn="urn:adsk.eagle:package:6644353/2"/>
+<part name="U$2" library="switches" deviceset="TVAF06-A020B-R" device=""/>
+<part name="GND12" library="supply1" library_urn="urn:adsk.eagle:library:371" deviceset="GND" device=""/>
 </parts>
 <sheets>
@@
 <attribute name="NAME" x="-76.2" y="44.45" size="1.778" layer="95" rot="R180"/>
 <attribute name="VALUE" x="-76.2" y="63.5" size="1.778" layer="95" rot="R180"/>
+</instance>
+<instance part="U$2" gate="G$1" x="-12.7" y="-40.64" smashed="yes" rot="R270">
+<attribute name="NAME" x="-10.16" y="-35.56" size="1.778" layer="95" rot="R270"/>
+<attribute name="VALUE" x="-17.78" y="-33.02" size="1.778" layer="96" rot="R270"/>
+</instance>
+<instance part="GND12" gate="1" x="-12.7" y="-50.8" smashed="yes">
+<attribute name="VALUE" x="-15.24" y="-53.34" size="1.778" layer="96"/>
 </instance>
 </instances>
@@
 <pinref part="LED" gate="G$1" pin="C"/>
 <pinref part="GND11" gate="1" pin="GND"/>
+</segment>
+<segment>
+<pinref part="U$2" gate="G$1" pin="B"/>
+<pinref part="GND12" gate="1" pin="GND"/>
 </segment>
 </net>
@@
 <pinref part="C7" gate="G$1" pin="1"/>
 <label x="-10.16" y="-33.02" size="1.778" layer="95" xref="yes"/>
-<wire x1="-27.94" y1="-33.02" x2="-10.16" y2="-33.02" width="0.1524" layer="91"/>
-</segment>
-</net>
+<wire x1="-27.94" y1="-33.02" x2="-12.7" y2="-33.02" width="0.1524" layer="91"/>
+<pinref part="U$2" gate="G$1" pin="A"/>
+<wire x1="-12.7" y1="-33.02" x2="-10.16" y2="-33.02" width="0.1524" layer="91"/>
+<junction x="-12.7" y="-33.02"/>
+</segment>
+</net>
